File: Schematic/WatchBorad/WatchBorad.sch (KiCad schematic (older format))
At the start: 0 parts

Commit message: Revert "Added connectors for top-board-schematic"
This reverts commit 6170a2acdf532fd042b1f8efa63f942ad96a6e4b.
Parts:
- added C1, C10, C11, C12, C13, C14, C16, C2, C3, C4, C7, C8, C9: 0.1uF, Capacitor_SMD:C_0805_2012Metric_Pad1.15x1.40mm_HandSolder, symbol Device:C
- added C15: 10nF, Capacitor_SMD:C_0805_2012Metric_Pad1.15x1.40mm_HandSolder, symbol Device:C
- added D1: LED, LED_SMD:LED_0805_2012Metric_Pad1.15x1.40mm_HandSolder, symbol Device:LED
- added F1: Polyfuse, Fuse:Fuse_1206_3216Metric_Pad1.42x1.75mm_HandSolder, symbol Device:Polyfuse
- added IC1: TXS0108E, TXS0108E:PW_R-PDSO-G20, symbol TXS0108E:TXS0108E
- added J1: Conn_01x06_Male, Connector_PinHeader_2.54mm:PinHeader_1x06_P2.54mm_Vertical, symbol Connector:Conn_01x06_Male
- added J2: Conn_01x09_Female, Connector_PinSocket_2.54mm:PinSocket_1x09_P2.54mm_Vertical, symbol Connector:Conn_01x09_Female
- added J3: USB_B_Mini, Connector_USB:USB_Mini-B_Lumberg_2486_01_Horizontal, symbol Connector:USB_B_Mini
- added J4: Conn_01x10_Female, Connector_PinSocket_2.54mm:PinSocket_1x10_P2.54mm_Vertical, symbol Connector:Conn_01x10_Female
- added J5: Conn_01x06_Female, Connector_PinSocket_2.54mm:PinSocket_1x06_P2.54mm_Vertical, symbol Connector:Conn_01x06_Female
- added J6: Conn_01x04_Male, Connector_PinHeader_2.54mm:PinHeader_1x04_P2.54mm_Vertical, symbol Connector:Conn_01x04_Male
- added J7, J8: Conn_01x11_Female, Connector_PinSocket_2.54mm:PinSocket_1x11_P2.54mm_Vertical, symbol Connector:Conn_01x11_Female
- added J9: Conn_01x12_Female, Connector_PinSocket_2.54mm:PinSocket_1x12_P2.54mm_Vertical, symbol Connector:Conn_01x12_Female
- added R1: 10K, Resistor_SMD:R_0805_2012Metric_Pad1.15x1.40mm_HandSolder, symbol Device:R
- added R2: R100, Resistor_SMD:R_0805_2012Metric_Pad1.15x1.40mm_HandSolder, symbol Device:R
- added R3: 1.5K, Resistor_SMD:R_0805_2012Metric_Pad1.15x1.40mm_HandSolder, symbol Device:R
- added R4, R5, R6: 4.7k, Resistor_SMD:R_0805_2012Metric_Pad1.15x1.40mm_HandSolder, symbol Device:R
- added R7: 3.3k, Resistor_SMD:R_0805_2012Metric_Pad1.15x1.40mm_HandSolder, symbol Device:R
- added R8, R9, R? (x2): 2k, Resistor_SMD:R_0805_2012Metric_Pad1.15x1.40mm_HandSolder, symbol Device:R
- added RESET1, SW1, SW2, SW? (x2): SW_Push, Button_Switch_SMD:SW_SPST_SKQG_WithStem, symbol Switch:SW_Push
- added U1: E73-2G4M04S-52832, RF_Module:E73-2G4M04S, symbol RF_Module:E73-2G4M04S-52832
- added U2: FH26-13S-0.3SHW(05), FH26W-13S-0:FH26-13S-0.3SHW(05), symbol Hirose_connectors:FH26-13S-0.3SHW(05)
- added U3: W25Q16BVSSIG, W25Q16BVSSIG:SOIC127P790X216-8N, symbol W25Q16BVSSIG:W25Q16BVSSIG
- added U4: LD1117S33TR_SOT223, Package_TO_SOT_SMD:SOT-223-3_TabPin2, symbol Regulator_Linear:LD1117S33TR_SOT223
- added U6: MCP1700-1802E_SOT23, Package_TO_SOT_SMD:SOT-23, symbol Regulator_Linear:MCP1700-1802E_SOT23
- added U7: LP2985-2.8, Package_TO_SOT_SMD:SOT-23-5, symbol Regulator_Linear:LP2985-2.8
- added U8: MPU-9250, QFN40P300X300X105-24N, symbol MPU-9250:MPU-9250
Connections:
- new net: IC1.10 (OE), R1.1
- new net: D1.2 (A), R3.2
- new net: C12.1, U7.4 (BP)
- new net: R?.2, SW?.2
- new net: R?.1, SW?.2
- new net: R6.2, U8.22 (~CS~)
- new net: F1.2, J3.1 (VBUS)
- new net: R8.2, SW1.2
- new net: R9.2, SW2.2
- new net +1V8: C11.1, C3.1, IC1.2 (VCCA), R1.2, U2.11, U6.2 (VO)
- new net +2V8: C4.1, U2.12, U7.5 (VOUT)
- new net +3V3: C1.1, C10.1, C13.1, C14.1, C15.1, C16.1, C2.1, C7.1, C8.1, IC1.19 (VCCB), J1.1 (Pin_1), J2.1 (Pin_1), J4.1 (Pin_1), J5.1 (Pin_1), J6.1 (Pin_1), R2.1, R4.1, R5.1, R6.1, R7.1, R8.1, R9.1, R?.1, R?.2, U1.16 (VCC), U3.3 (/WP(IO2)), U3.7 (/HOLD(IO3)), U3.8 (VCC), U4.2 (VO), U6.3 (VI), U7.1 (VIN), U7.3 (ON/~OFF~), U8.1 (RESV_1), U8.10 (REGOUT), U8.13 (VDD), U8.8 (VDDIO)
- new net +5V: C9.1, F1.1, U4.3 (VI)
- new net BRD_LED_P13: R3.1, U1.28 (P0.13)
- new net CS_1.8: IC1.5 (A4), U2.9
- new net DISP_CS: IC1.16 (B4), J2.7 (Pin_7), J7.7 (Pin_7), U1.10 (AIN6/P0.30)
- new net DISP_FMARK: IC1.15 (B5), J2.6 (Pin_6), J7.6 (Pin_6), U1.9 (AIN5/P0.29)
- new net DISP_RESET: IC1.17 (B3), J2.8 (Pin_8), J7.8 (Pin_8), U1.11 (AIN7/P0.31)
- new net DISP_RS: IC1.12 (B8), J2.3 (Pin_3), J7.3 (Pin_3), U1.6 (P0.26)
- new net DISP_SCLK: IC1.14 (B6), J2.5 (Pin_5), J7.5 (Pin_5), U1.8 (AIN4/P0.28)
- new net DISP_SDA: IC1.13 (B7), J2.4 (Pin_4), J7.4 (Pin_4), U1.7 (P0.27)
- new net FLASH_CS: J5.2 (Pin_2), U3.1 (/CS)
- new net FLASH_MISO: J5.3 (Pin_3), U3.2 (DO(IO1))
- new net FLASH_MOSI: J5.6 (Pin_6), U3.5 (DI(IO0))
- new net FLASH_SCK: J5.5 (Pin_5), U3.6 (CLK)
- new net FMARK_1.8: IC1.6 (A5), U2.5
- new net GND: C1.2, C10.2, C11.2, C12.2, C13.2, C14.2, C15.2, C16.2, C2.2, C3.2, C4.2, C7.2, C8.2, C9.2, D1.1 (K), IC1.11 (GND), J1.2 (Pin_2), J2.2 (Pin_2), J3.5 (GND), J3.6 (Shield), J4.2 (Pin_2), J5.4 (Pin_4), J6.4 (Pin_4), RESET1.2, SW1.1, SW2.1, SW?.1, SW?.1, U1.0 (GND), U1.1 (GND), U1.15 (GND), U1.2 (GND), U1.42 (GND), U1.43 (GND), U2.1, U2.13, U2.2, U2.4, U3.4 (GND), U4.1 (GND), U6.1 (GND), U7.2 (GND), U8.18 (GND), U8.20 (RESV_20)
- new net LEDA: R2.2, U2.3
- new net MPU_ADO: J4.7 (Pin_7), U8.9 (AD0/SDO)
- new net MPU_INT: J4.8 (Pin_8), R7.2, U8.12 (INT)
- new net MPU_SCLK: J4.3 (Pin_3), R4.2, U8.23 (SCL/SCLK)
- new net MPU_SDA: J4.4 (Pin_4), R5.2, U8.24 (SDA/SDI)
- new net MPU_SYNC: J4.10 (Pin_10), U8.11 (FSYNC)
- new net P_05: J7.2 (Pin_2), U1.5 (P0.25)
- new net P_DCC: J7.10 (Pin_10), U1.13 (DCC)
- new net P_DEC1: J7.11 (Pin_11), U1.14 (DEC1)
- new net P_DEC2: U1.3 (DEC2)
- new net P_DEC3: J7.1 (Pin_1), U1.4 (DEC3)
- new net P_DEC4: J7.9 (Pin_9), U1.12 (DEC4)
- new net RESET_1.8: IC1.4 (A3), U2.10
- new net RS_1.8: IC1.9 (A8), U2.7
- new net SCLK_1.8: IC1.7 (A6), U2.8
- new net SDA_1.8: IC1.8 (A7), U2.6
- new net SWD_RESET: J1.5 (Pin_5), RESET1.1, U1.36 (P0.21/~RESET)
- new net SWD_SWDCLK: J1.4 (Pin_4), U1.37 (SWDCLK)
- new net SWD_SWDIO: J1.3 (Pin_3), U1.38 (SWDIO)
- new net SWD_SWO: J1.6 (Pin_6), U1.33 (SWO/P0.18)
- new net UART1_RX: J6.3 (Pin_3)
- new net UART1_TX: J6.2 (Pin_2)
Other:
- note added: "Diplsay & board supply"
- note added: "Display module, Controller ST7789V"
- note added: "Gyroscope & Accelerometer & Magnetometer with I2C interface"
- note added: "MCU Reset"
- note added: "NRF52832-E73 Module"
- note added: "Onboard RED LED"
- note added: "SPI FLASH Memory\n"
- note added: "SWD programming interface"
- note added: "UART1"
- note added: "USB Supply"
- note added: "User Buttons"
