File: Schematic/WatchBorad/PSU_logic.sch (KiCad schematic (older format))
At the start: 30 parts, among them J4 TYPE-C-31-M-17, SW1 SW_Push, SW2 SW_Push, U5 BQ21040DBVT, U6 STC3100IQT, U7 max16054azt+t, U8 TPS2115APWR

Commit message: PBs are modified to one logic. Some minot changes
Parts:
- added C23, C27, C28: 10 uF, Capacitors_SMD:C_0603_HandSoldering, symbol Device:C
- added C26: 100 nF, Capacitors_SMD:C_0603_HandSoldering, symbol Device:C
- C24: value 1 uF 16V -> 10 uF; LCSC https://lcsc.com/product-detail/Multilayer-Ceramic-Capacitors-MLCC-SMD-SMT_SANYEAR-C0603X5R105K160NT_C475249.html -> https://lcsc.com/product-detail/Multilayer-Ceramic-Capacitors-MLCC-SMD-SMT_SANYEAR-C0603X5R106M160NT_C466781.html
- C25: value 1 uF 16V -> 100 nF; LCSC https://lcsc.com/product-detail/Multilayer-Ceramic-Capacito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 -> (none)
- renumbered C26 to C29, C27 to C30, C28 to C31, J4 to J3, R9 to R15, R10 to R16, R11 to R17, R12 to R18, R13 to R19, R14 to R20, R15 to R21, R16 to R22, R17 to R23, R18 to R24, R19 to R25, TP6 to TP11, TP7 to TP12
Connections:
- net +5V: now also C24.1, C28.1; no longer C25.1
- net +BATT: now also C23.1, C27.1; no longer C24.1
- net GND: now also C26.2, C27.2, C28.2
- net V_Battery_N: now also C23.2
- net at R15.1, R18.2, SW2.1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: now also C26.1
- net at R16.1, R17.2, SW1.1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: now also C25.1
Other:
- note added: "1.5A\n"
- note added: "D1| D0 | VI(IN2) > VI(IN1) | OUT\n0 |1 |No |IN1\n0 |1 |Yes |IN2"
- moved on the sheet: D1, J3, R15, R16

Commit message: Fixed LCSC schematic link :Schematic [SCHEMATIC]
Parts:
- C23, C24, C27, C28: LCSC https://lcsc.com/product-detail/Multilayer-Ceramic-Capacito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 -> (none); lcsc (none) -> https://lcsc.com/product-detail/Multilayer-Ceramic-Capacito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
Changed lines of the file:
@@
 F 2 "Capacitors_SMD:C_0603_HandSoldering" H 1663 6400 50  0001 C CNN
 F 3 "~" H 1625 6550 50  0001 C CNN
-F 4 "https://lcsc.com/product-detail/Multilayer-Ceramic-Capacitors-MLCC-SMD-SMT_SANYEAR-C0603X5R106M160NT_C466781.html" H 1625 6550 50  0001 C CNN "LCSC"
+F 4 "" H 1625 6550 50  0001 C CNN "LCSC"
+F 5 "https://lcsc.com/product-detail/Multilayer-Ceramic-Capacitors-MLCC-SMD-SMT_SANYEAR-C0603X5R106M160NT_C466781.html" H 1625 6550 50  0001 C CNN "lcsc"
 	1    1625 6550
 	1    0    0    -1
@@
 F 2 "Capacitors_SMD:C_0603_HandSoldering" H 1813 4400 50  0001 C CNN
 F 3 "~" H 1775 4550 50  0001 C CNN
-F 4 "https://lcsc.com/product-detail/Multilayer-Ceramic-Capacitors-MLCC-SMD-SMT_SANYEAR-C0603X5R106M160NT_C466781.html" H 1775 4550 50  0001 C CNN "LCSC"
+F 4 "" H 1775 4550 50  0001 C CNN "LCSC"
+F 5 "https://lcsc.com/product-detail/Multilayer-Ceramic-Capacitors-MLCC-SMD-SMT_SANYEAR-C0603X5R106M160NT_C466781.html" H 1775 4550 50  0001 C CNN "lcsc"
 	1    1775 4550
 	1    0    0    -1
@@
 F 2 "Capacitors_SMD:C_0603_HandSoldering" H 3013 6725 50  0001 C CNN
 F 3 "~" H 2975 6875 50  0001 C CNN
-F 4 "https://lcsc.com/product-detail/Multilayer-Ceramic-Capacitors-MLCC-SMD-SMT_SANYEAR-C0603X5R106M160NT_C466781.html" H 2975 6875 50  0001 C CNN "LCSC"
+F 4 "" H 2975 6875 50  0001 C CNN "LCSC"
+F 5 "https://lcsc.com/product-detail/Multilayer-Ceramic-Capacitors-MLCC-SMD-SMT_SANYEAR-C0603X5R106M160NT_C466781.html" H 2975 6875 50  0001 C CNN "lcsc"
 	1    2975 6875
 	1    0    0    -1
@@
 F 2 "Capacitors_SMD:C_0603_HandSoldering" H 3388 4225 50  0001 C CNN
 F 3 "~" H 3350 4375 50  0001 C CNN
-F 4 "https://lcsc.com/product-detail/Multilayer-Ceramic-Capacitors-MLCC-SMD-SMT_SANYEAR-C0603X5R106M160NT_C466781.html" H 3350 4375 50  0001 C CNN "LCSC"
+F 4 "" H 3350 4375 50  0001 C CNN "LCSC"
+F 5 "https://lcsc.com/product-detail/Multilayer-Ceramic-Capacitors-MLCC-SMD-SMT_SANYEAR-C0603X5R106M160NT_C466781.html" H 3350 4375 50  0001 C CNN "lcsc"
 	1    3350 4375
 	1    0    0    -1

Commit message: Fixed components references for 0603 resistors and capacitors[SCHEMATIC]
Parts:
- C23, C24, C25, C26, C27, C28, C29, C30, C31: footprint Capacitors_SMD:C_0603_HandSoldering -> Capacitor_SMD:C_0603_1608Metric_Pad1.08x0.95mm_HandSolder
- R15, R16, R17, R18, R19, R20, R21, R22, R23, R24, R25: footprint Resistors_SMD:R_0603_HandSoldering -> Resistor_SMD:R_0603_1608Metric_Pad0.98x0.95mm_HandSolder
Changed lines of the file:
@@
 F 0 "C29" H 5450 2675 50  0000 L CNN
 F 1 "100 nF" V 5275 2475 50  0000 L CNN
-F 2 "Capacitors_SMD:C_0603_HandSoldering" H 5463 2450 50  0001 C CNN
+F 2 "Capacitor_SMD:C_0603_1608Metric_Pad1.08x0.95mm_HandSolder" H 5463 2450 50  0001 C CNN
 F 3 "~" H 5425 2600 50  0001 C CNN
 	1    5425 2600
@@
 F 0 "R25" H 8095 1196 50  0000 L CNN
 F 1 "10k" H 8095 1105 50  0000 L CNN
-F 2 "Resistors_SMD:R_0603_HandSoldering" V 7955 1150 50  0001 C CNN
+F 2 "Resistor_SMD:R_0603_1608Metric_Pad0.98x0.95mm_HandSolder" V 7955 1150 50  0001 C CNN
 F 3 "~" H 8025 1150 50  0001 C CNN
 	1    8025 1150
@@
 F 0 "R21" V 4975 1575 50  0000 L CNN
 F 1 "10k" V 4975 1875 50  0000 L CNN
-F 2 "Resistors_SMD:R_0603_HandSoldering" V 5005 1775 50  0001 C CNN
+F 2 "Resistor_SMD:R_0603_1608Metric_Pad0.98x0.95mm_HandSolder" V 5005 1775 50  0001 C CNN
 F 3 "~" H 5075 1775 50  0001 C CNN
 	1    5075 1775
@@
 F 0 "R17" H 3150 2550 50  0000 L CNN
 F 1 "10k" H 3100 2650 50  0000 L CNN
-F 2 "Resistors_SMD:R_0603_HandSoldering" V 2955 2575 50  0001 C CNN
+F 2 "Resistor_SMD:R_0603_1608Metric_Pad0.98x0.95mm_HandSolder" V 2955 2575 50  0001 C CNN
 F 3 "~" H 3025 2575 50  0001 C CNN
 	1    3025 2575
@@
 F 0 "R18" H 3000 1850 50  0000 L CNN
 F 1 "10k" H 3000 1975 50  0000 L CNN
-F 2 "Resistors_SMD:R_0603_HandSoldering" V 3130 1900 50  0001 C CNN
+F 2 "Resistor_SMD:R_0603_1608Metric_Pad0.98x0.95mm_HandSolder" V 3130 1900 50  0001 C CNN
 F 3 "~" H 3200 1900 50  0001 C CNN
 	1    3200 1900
@@
 F 0 "R24" V 7043 4925 50  0000 C CNN
 F 1 "330" V 7134 4925 50  0000 C CNN
-F 2 "Resistors_SMD:R_0603_HandSoldering" V 7180 4925 50  0001 C CNN
+F 2 "Resistor_SMD:R_0603_1608Metric_Pad0.98x0.95mm_HandSolder" V 7180 4925 50  0001 C CNN
 F 3 "https://lcsc.com/product-detail/Others_Viking-Tech-ARG03FTC3300_C217969.html" H 7250 4925 50  0001 C CNN
 	1    7250 4925
@@
 F 0 "C30" H 6500 4700 50  0000 L CNN
 F 1 "100 nF" V 6325 4500 50  0000 L CNN
-F 2 "Capacitors_SMD:C_0603_HandSoldering" H 6513 4475 50  0001 C CNN
+F 2 "Capacitor_SMD:C_0603_1608Metric_Pad1.08x0.95mm_HandSolder" H 6513 4475 50  0001 C CNN
 F 3 "~" H 6475 4625 50  0001 C CNN
 	1    6475 4625
@@
 F 0 "C31" H 7100 4700 50  0000 L CNN
 F 1 "100 nF" V 6950 4450 50  0000 L CNN
-F 2 "Capacitors_SMD:C_0603_HandSoldering" H 7113 4475 50  0001 C CNN
+F 2 "Capacitor_SMD:C_0603_1608Metric_Pad1.08x0.95mm_HandSolder" H 7113 4475 50  0001 C CNN
 F 3 "~" H 7075 4625 50  0001 C CNN
 	1    7075 4625
@@
 F 0 "R20" V 3600 4625 50  0000 L CNN
 F 1 "10k" V 3450 4600 50  0000 L CNN
-F 2 "Resistors_SMD:R_0603_HandSoldering" V 3455 4675 50  0001 C CNN
+F 2 "Resistor_SMD:R_0603_1608Metric_Pad0.98x0.95mm_HandSolder" V 3455 4675 50  0001 C CNN
 F 3 "~" H 3525 4675 50  0001 C CNN
 	1    3525 4675
@@
 F 0 "R23" H 5575 4600 50  0000 L CNN
 F 1 "10k" V 5875 4550 50  0000 L CNN
-F 2 "Resistors_SMD:R_0603_HandSoldering" V 5730 4625 50  0001 C CNN
+F 2 "Resistor_SMD:R_0603_1608Metric_Pad0.98x0.95mm_HandSolder" V 5730 4625 50  0001 C CNN
 F 3 "~" H 5800 4625 50  0001 C CNN
 	1    5800 4625
@@
 F 0 "R22" V 5125 6275 50  0000 L CNN
 F 1 "200k 0.1%" V 5200 6125 50  0000 L CNN
-F 2 "Resistors_SMD:R_0603_HandSoldering" V 5230 6325 50  0001 C CNN
+F 2 "Resistor_SMD:R_0603_1608Metric_Pad0.98x0.95mm_HandSolder" V 5230 6325 50  0001 C CNN
 F 3 "~" H 5300 6325 50  0001 C CNN
 	1    5300 6325
@@
 F 0 "R19" H 3475 6800 50  0000 L CNN
 F 1 "0.15 Ohm" V 3300 6675 50  0000 L CNN
-F 2 "Resistors_SMD:R_0603_HandSoldering" V 3330 6850 50  0001 C CNN
+F 2 "Resistor_SMD:R_0603_1608Metric_Pad0.98x0.95mm_HandSolder" V 3330 6850 50  0001 C CNN
 F 3 "~" H 3400 6850 50  0001 C CNN
 F 4 "https://lcsc.com/product-detail/Chip-Resistor-Surface-Mount_UNI-ROYAL-Uniroyal-Elec-0603WAF150LT5E_C45879.html" V 3400 6850 50  0001 C CNN "lcsc"
@@
 F 0 "R15" V 1843 1650 50  0000 C CNN
 F 1 "330" V 1934 1650 50  0000 C CNN
-F 2 "Resistors_SMD:R_0603_HandSoldering" V 1980 1650 50  0001 C CNN
+F 2 "Resistor_SMD:R_0603_1608Metric_Pad0.98x0.95mm_HandSolder" V 1980 1650 50  0001 C CNN
 F 3 "https://lcsc.com/product-detail/Others_Viking-Tech-ARG03FTC3300_C217969.html" H 2050 1650 50  0001 C CNN
 	1    2050 1650
@@
 F 0 "R16" V 1843 2275 50  0000 C CNN
 F 1 "330" V 1934 2275 50  0000 C CNN
-F 2 "Resistors_SMD:R_0603_HandSoldering" V 1980 2275 50  0001 C CNN
+F 2 "Resistor_SMD:R_0603_1608Metric_Pad0.98x0.95mm_HandSolder" V 1980 2275 50  0001 C CNN
 F 3 "https://lcsc.com/product-detail/Others_Viking-Tech-ARG03FTC3300_C217969.html" H 2050 2275 50  0001 C CNN
 	1    2050 2275
@@
 F 0 "C23" H 1650 6625 50  0000 L CNN
 F 1 "10 uF" V 1475 6425 50  0000 L CNN
-F 2 "Capacitors_SMD:C_0603_HandSoldering" H 1663 6400 50  0001 C CNN
+F 2 "Capacitor_SMD:C_0603_1608Metric_Pad1.08x0.95mm_HandSolder" H 1663 6400 50  0001 C CNN
 F 3 "~" H 1625 6550 50  0001 C CNN
 F 4 "" H 1625 6550 50  0001 C CNN "LCSC"
@@
 F 0 "C24" H 1800 4625 50  0000 L CNN
 F 1 "10 uF" V 1625 4425 50  0000 L CNN
-F 2 "Capacitors_SMD:C_0603_HandSoldering" H 1813 4400 50  0001 C CNN
+F 2 "Capacitor_SMD:C_0603_1608Metric_Pad1.08x0.95mm_HandSolder" H 1813 4400 50  0001 C CNN
 F 3 "~" H 1775 4550 50  0001 C CNN
 F 4 "" H 1775 4550 50  0001 C CNN "LCSC"
@@
 F 0 "C27" H 3000 6950 50  0000 L CNN
 F 1 "10 uF" V 2825 6750 50  0000 L CNN
-F 2 "Capacitors_SMD:C_0603_HandSoldering" H 3013 6725 50  0001 C CNN
+F 2 "Capacitor_SMD:C_0603_1608Metric_Pad1.08x0.95mm_HandSolder" H 3013 6725 50  0001 C CNN
 F 3 "~" H 2975 6875 50  0001 C CNN
 F 4 "" H 2975 6875 50  0001 C CNN "LCSC"
@@
 F 0 "C28" H 3375 4450 50  0000 L CNN
 F 1 "10 uF" V 3200 4250 50  0000 L CNN
-F 2 "Capacitors_SMD:C_0603_HandSoldering" H 3388 4225 50  0001 C CNN
+F 2 "Capacitor_SMD:C_0603_1608Metric_Pad1.08x0.95mm_HandSolder" H 3388 4225 50  0001 C CNN
 F 3 "~" H 3350 4375 50  0001 C CNN
 F 4 "" H 3350 4375 50  0001 C CNN "LCSC"
@@
 F 0 "C25" H 2325 2600 50  0000 L CNN
 F 1 "100 nF" V 2175 2350 50  0000 L CNN
-F 2 "Capacitors_SMD:C_0603_HandSoldering" H 2338 2375 50  0001 C CNN
+F 2 "Capacitor_SMD:C_0603_1608Metric_Pad1.08x0.95mm_HandSolder" H 2338 2375 50  0001 C CNN
 F 3 "~" H 2300 2525 50  0001 C CNN
 	1    2300 2525
@@
 F 0 "C26" H 2625 2600 50  0000 L CNN
 F 1 "100 nF" V 2475 2350 50  0000 L CNN
-F 2 "Capacitors_SMD:C_0603_HandSoldering" H 2638 2375 50  0001 C CNN
+F 2 "Capacitor_SMD:C_0603_1608Metric_Pad1.08x0.95mm_HandSolder" H 2638 2375 50  0001 C CNN
 F 3 "~" H 2600 2525 50  0001 C CNN
 	1    2600 2525

Commit message: Updated 0603 components from hand-solder version to fabrical
Parts:
- C23, C24, C25, C26, C27, C28, C29, C30, C31: footprint Capacitor_SMD:C_0603_1608Metric_Pad1.08x0.95mm_HandSolder -> Capacitor_SMD:C_0603_1608Metric
- R15, R16, R17, R18, R19, R20, R21, R22, R23, R24, R25: footprint Resistor_SMD:R_0603_1608Metric_Pad0.98x0.95mm_HandSolder -> Resistor_SMD:R_0603_1608Metric
Changed lines of the file:
@@
 F 0 "C29" H 5450 2675 50  0000 L CNN
 F 1 "100 nF" V 5275 2475 50  0000 L CNN
-F 2 "Capacitor_SMD:C_0603_1608Metric_Pad1.08x0.95mm_HandSolder" H 5463 2450 50  0001 C CNN
+F 2 "Capacitor_SMD:C_0603_1608Metric" H 5463 2450 50  0001 C CNN
 F 3 "~" H 5425 2600 50  0001 C CNN
 	1    5425 2600
@@
 F 0 "R25" H 8095 1196 50  0000 L CNN
 F 1 "10k" H 8095 1105 50  0000 L CNN
-F 2 "Resistor_SMD:R_0603_1608Metric_Pad0.98x0.95mm_HandSolder" V 7955 1150 50  0001 C CNN
+F 2 "Resistor_SMD:R_0603_1608Metric" V 7955 1150 50  0001 C CNN
 F 3 "~" H 8025 1150 50  0001 C CNN
 	1    8025 1150
@@
 F 0 "R21" V 4975 1575 50  0000 L CNN
 F 1 "10k" V 4975 1875 50  0000 L CNN
-F 2 "Resistor_SMD:R_0603_1608Metric_Pad0.98x0.95mm_HandSolder" V 5005 1775 50  0001 C CNN
+F 2 "Resistor_SMD:R_0603_1608Metric" V 5005 1775 50  0001 C CNN
 F 3 "~" H 5075 1775 50  0001 C CNN
 	1    5075 1775
@@
 F 0 "R17" H 3150 2550 50  0000 L CNN
 F 1 "10k" H 3100 2650 50  0000 L CNN
-F 2 "Resistor_SMD:R_0603_1608Metric_Pad0.98x0.95mm_HandSolder" V 2955 2575 50  0001 C CNN
+F 2 "Resistor_SMD:R_0603_1608Metric" V 2955 2575 50  0001 C CNN
 F 3 "~" H 3025 2575 50  0001 C CNN
 	1    3025 2575
@@
 F 0 "R18" H 3000 1850 50  0000 L CNN
 F 1 "10k" H 3000 1975 50  0000 L CNN
-F 2 "Resistor_SMD:R_0603_1608Metric_Pad0.98x0.95mm_HandSolder" V 3130 1900 50  0001 C CNN
+F 2 "Resistor_SMD:R_0603_1608Metric" V 3130 1900 50  0001 C CNN
 F 3 "~" H 3200 1900 50  0001 C CNN
 	1    3200 1900
@@
 F 0 "R24" V 7043 4925 50  0000 C CNN
 F 1 "330" V 7134 4925 50  0000 C CNN
-F 2 "Resistor_SMD:R_0603_1608Metric_Pad0.98x0.95mm_HandSolder" V 7180 4925 50  0001 C CNN
+F 2 "Resistor_SMD:R_0603_1608Metric" V 7180 4925 50  0001 C CNN
 F 3 "https://lcsc.com/product-detail/Others_Viking-Tech-ARG03FTC3300_C217969.html" H 7250 4925 50  0001 C CNN
 	1    7250 4925
@@
 F 0 "C30" H 6500 4700 50  0000 L CNN
 F 1 "100 nF" V 6325 4500 50  0000 L CNN
-F 2 "Capacitor_SMD:C_0603_1608Metric_Pad1.08x0.95mm_HandSolder" H 6513 4475 50  0001 C CNN
+F 2 "Capacitor_SMD:C_0603_1608Metric" H 6513 4475 50  0001 C CNN
 F 3 "~" H 6475 4625 50  0001 C CNN
 	1    6475 4625
@@
 F 0 "C31" H 7100 4700 50  0000 L CNN
 F 1 "100 nF" V 6950 4450 50  0000 L CNN
-F 2 "Capacitor_SMD:C_0603_1608Metric_Pad1.08x0.95mm_HandSolder" H 7113 4475 50  0001 C CNN
+F 2 "Capacitor_SMD:C_0603_1608Metric" H 7113 4475 50  0001 C CNN
 F 3 "~" H 7075 4625 50  0001 C CNN
 	1    7075 4625
@@
 F 0 "R20" V 3600 4625 50  0000 L CNN
 F 1 "10k" V 3450 4600 50  0000 L CNN
-F 2 "Resistor_SMD:R_0603_1608Metric_Pad0.98x0.95mm_HandSolder" V 3455 4675 50  0001 C CNN
+F 2 "Resistor_SMD:R_0603_1608Metric" V 3455 4675 50  0001 C CNN
 F 3 "~" H 3525 4675 50  0001 C CNN
 	1    3525 4675
@@
 F 0 "R23" H 5575 4600 50  0000 L CNN
 F 1 "10k" V 5875 4550 50  0000 L CNN
-F 2 "Resistor_SMD:R_0603_1608Metric_Pad0.98x0.95mm_HandSolder" V 5730 4625 50  0001 C CNN
+F 2 "Resistor_SMD:R_0603_1608Metric" V 5730 4625 50  0001 C CNN
 F 3 "~" H 5800 4625 50  0001 C CNN
 	1    5800 4625
@@
 F 0 "R22" V 5125 6275 50  0000 L CNN
 F 1 "200k 0.1%" V 5200 6125 50  0000 L CNN
-F 2 "Resistor_SMD:R_0603_1608Metric_Pad0.98x0.95mm_HandSolder" V 5230 6325 50  0001 C CNN
+F 2 "Resistor_SMD:R_0603_1608Metric" V 5230 6325 50  0001 C CNN
 F 3 "~" H 5300 6325 50  0001 C CNN
 	1    5300 6325
@@
 F 0 "R19" H 3475 6800 50  0000 L CNN
 F 1 "0.15 Ohm" V 3300 6675 50  0000 L CNN
-F 2 "Resistor_SMD:R_0603_1608Metric_Pad0.98x0.95mm_HandSolder" V 3330 6850 50  0001 C CNN
+F 2 "Resistor_SMD:R_0603_1608Metric" V 3330 6850 50  0001 C CNN
 F 3 "~" H 3400 6850 50  0001 C CNN
 F 4 "https://lcsc.com/product-detail/Chip-Resistor-Surface-Mount_UNI-ROYAL-Uniroyal-Elec-0603WAF150LT5E_C45879.html" V 3400 6850 50  0001 C CNN "lcsc"
@@
 F 0 "R15" V 1843 1650 50  0000 C CNN
 F 1 "330" V 1934 1650 50  0000 C CNN
-F 2 "Resistor_SMD:R_0603_1608Metric_Pad0.98x0.95mm_HandSolder" V 1980 1650 50  0001 C CNN
+F 2 "Resistor_SMD:R_0603_1608Metric" V 1980 1650 50  0001 C CNN
 F 3 "https://lcsc.com/product-detail/Others_Viking-Tech-ARG03FTC3300_C217969.html" H 2050 1650 50  0001 C CNN
 	1    2050 1650
@@
 F 0 "R16" V 1843 2275 50  0000 C CNN
 F 1 "330" V 1934 2275 50  0000 C CNN
-F 2 "Resistor_SMD:R_0603_1608Metric_Pad0.98x0.95mm_HandSolder" V 1980 2275 50  0001 C CNN
+F 2 "Resistor_SMD:R_0603_1608Metric" V 1980 2275 50  0001 C CNN
 F 3 "https://lcsc.com/product-detail/Others_Viking-Tech-ARG03FTC3300_C217969.html" H 2050 2275 50  0001 C CNN
 	1    2050 2275
@@
 F 0 "C23" H 1650 6625 50  0000 L CNN
 F 1 "10 uF" V 1475 6425 50  0000 L CNN
-F 2 "Capacitor_SMD:C_0603_1608Metric_Pad1.08x0.95mm_HandSolder" H 1663 6400 50  0001 C CNN
+F 2 "Capacitor_SMD:C_0603_1608Metric" H 1663 6400 50  0001 C CNN
 F 3 "~" H 1625 6550 50  0001 C CNN
 F 4 "" H 1625 6550 50  0001 C CNN "LCSC"
@@
 F 0 "C24" H 1800 4625 50  0000 L CNN
 F 1 "10 uF" V 1625 4425 50  0000 L CNN
-F 2 "Capacitor_SMD:C_0603_1608Metric_Pad1.08x0.95mm_HandSolder" H 1813 4400 50  0001 C CNN
+F 2 "Capacitor_SMD:C_0603_1608Metric" H 1813 4400 50  0001 C CNN
 F 3 "~" H 1775 4550 50  0001 C CNN
 F 4 "" H 1775 4550 50  0001 C CNN "LCSC"
@@
 F 0 "C27" H 3000 6950 50  0000 L CNN
 F 1 "10 uF" V 2825 6750 50  0000 L CNN
-F 2 "Capacitor_SMD:C_0603_1608Metric_Pad1.08x0.95mm_HandSolder" H 3013 6725 50  0001 C CNN
+F 2 "Capacitor_SMD:C_0603_1608Metric" H 3013 6725 50  0001 C CNN
 F 3 "~" H 2975 6875 50  0001 C CNN
 F 4 "" H 2975 6875 50  0001 C CNN "LCSC"
@@
 F 0 "C28" H 3375 4450 50  0000 L CNN
 F 1 "10 uF" V 3200 4250 50  0000 L CNN
-F 2 "Capacitor_SMD:C_0603_1608Metric_Pad1.08x0.95mm_HandSolder" H 3388 4225 50  0001 C CNN
+F 2 "Capacitor_SMD:C_0603_1608Metric" H 3388 4225 50  0001 C CNN
 F 3 "~" H 3350 4375 50  0001 C CNN
 F 4 "" H 3350 4375 50  0001 C CNN "LCSC"
@@
 F 0 "C25" H 2325 2600 50  0000 L CNN
 F 1 "100 nF" V 2175 2350 50  0000 L CNN
-F 2 "Capacitor_SMD:C_0603_1608Metric_Pad1.08x0.95mm_HandSolder" H 2338 2375 50  0001 C CNN
+F 2 "Capacitor_SMD:C_0603_1608Metric" H 2338 2375 50  0001 C CNN
 F 3 "~" H 2300 2525 50  0001 C CNN
 	1    2300 2525
@@
 F 0 "C26" H 2625 2600 50  0000 L CNN
 F 1 "100 nF" V 2475 2350 50  0000 L CNN
-F 2 "Capacitor_SMD:C_0603_1608Metric_Pad1.08x0.95mm_HandSolder" H 2638 2375 50  0001 C CNN
+F 2 "Capacitor_SMD:C_0603_1608Metric" H 2638 2375 50  0001 C CNN
 F 3 "~" H 2600 2525 50  0001 C CNN
 	1    2600 2525

Commit message: Updated parts list accroding to the Ruslan fixes
Parts:
- D1: footprint (none) -> LocalFootprints:TVS_DFN1006; lcsc https://lcsc.com/product-detail/TVS_PN-SILICON-PESDU0521P1_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 -> https://lcsc.com/product-detail/TVS_Leiditech-ESDA05CP_C384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
- SW1, SW2: footprint Buttons_Switches_SMD:SW_SPST_B3U-3000P-B -> OmronSwitch:SW_B3U-3000P; lcsc https://lcsc.com/products/Tactile-Switches_427.html?q=b3u-3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 -> https://lcsc.com/product-detail/Tactile-Switches_Omron-Elec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
Changed lines of the file:
@@
 F 0 "SW2" V 3050 1350 50  0000 C CNN
 F 1 "SW_Push" H 3050 1000 50  0000 C CNN
-F 2 "Buttons_Switches_SMD:SW_SPST_B3U-3000P-B" H 3050 1275 50  0001 C CNN
-F 3 "https://datasheet.lcsc.com/szlcsc/Omron-Electronics-B3U-3000PM-B_C306884.pdf" H 3050 1275 50  0001 C CNN
-F 4 "https://lcsc.com/products/Tactile-Switches_427.html?q=b3u-3000" H 3050 1075 50  0001 C CNN "lcsc"
+F 2 "OmronSwitch:SW_B3U-3000P" H 3050 1275 50  0001 C CNN
+F 3 "https://datasheet.lcsc.com/lcsc/2012042009_Omron-Electronics-B3U-3000P_C963349.pdf" H 3050 1275 50  0001 C CNN
+F 4 "https://lcsc.com/product-detail/Tactile-Switches_Omron-Electronics-B3U-3000P_C963349.html" H 3050 1075 50  0001 C CNN "lcsc"
 	1    3050 1075
 	0    -1   -1   0
@@
 F 0 "SW1" V 2925 2125 50  0000 C CNN
 F 1 "SW_Push" H 2875 1900 50  0000 C CNN
-F 2 "Buttons_Switches_SMD:SW_SPST_B3U-3000P-B" H 2875 2150 50  0001 C CNN
-F 3 "https://datasheet.lcsc.com/szlcsc/Omron-Electronics-B3U-3000PM-B_C306884.pdf" H 2875 2150 50  0001 C CNN
-F 4 "https://lcsc.com/products/Tactile-Switches_427.html?q=b3u-3000" H 2875 1950 50  0001 C CNN "lcsc"
+F 2 "OmronSwitch:SW_B3U-3000P" H 2875 2150 50  0001 C CNN
+F 3 "https://datasheet.lcsc.com/lcsc/2012042009_Omron-Electronics-B3U-3000P_C963349.pdf" H 2875 2150 50  0001 C CNN
+F 4 "https://lcsc.com/product-detail/Tactile-Switches_Omron-Electronics-B3U-3000P_C963349.html" H 2875 1950 50  0001 C CNN "lcsc"
 	1    2875 1950
 	0    -1   -1   0
@@
 F 0 "D1" V 1229 4604 50  0000 L CNN
 F 1 "D_TVS" V 1320 4604 50  0000 L CNN
-F 2 "" H 1275 4525 50  0001 C CNN
-F 3 "https://datasheet.lcsc.com/szlcsc/2003282109_PN-SILICON-PESDU0521P1_C499647.pdf" H 1275 4525 50  0001 C CNN
-F 4 "https://lcsc.com/product-detail/TVS_PN-SILICON-PESDU0521P1_C499647.html" V 1275 4525 50  0001 C CNN "lcsc"
+F 2 "LocalFootprints:TVS_DFN1006" H 1275 4525 50  0001 C CNN
+F 3 "https://datasheet.lcsc.com/lcsc/2012141705_Leiditech-ESDA05CP_C384839.pdf" H 1275 4525 50  0001 C CNN
+F 4 "https://lcsc.com/product-detail/TVS_Leiditech-ESDA05CP_C384839.html" V 1275 4525 50  0001 C CNN "lcsc"
 	1    1275 4525
 	0    1    1    0
