File: Schematic/WatchBorad/WatchBorad.kicad_pcb (KiCad board)
At the start: 4 copper layers, 35 x 35 mm, 118 parts, among them J1 Conn_01x07_Female, J3 TYPE-C-31-M-17, M1 Motor_DC, SW1 SW_Push, SW2 SW_Push, SW3 SW_Push, SW4 SW_Push, SW5 SW_Push, U1 LSM6DSLTR, U10 TPS62740DSST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

Commit message: Added cooper region for GND layer
Routing:
- added copper zone on In2.Cu, net GND
Changed lines of the file:
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@@
     (0 F.Cu signal)
     (1 In1.Cu power)
-    (2 In2.Cu power hide)
+    (2 In2.Cu power)
     (31 B.Cu signal)
     (32 B.Adhes user hide)
@@
   (segment (start 80.55 78.5) (end 80.7 78.65) (width 0.15) (layer B.Cu) (net 82))
   (segment (start 79.8 78.5) (end 80.55 78.5) (width 0.15) (layer B.Cu) (net 82))
-  (zone (net 0) (net_name "") (layer B.Cu) (hatch edge 0.508)
+  (zone (net 0) (net_name "") (layers F.Cu In1.Cu In2.Cu B.Cu) (hatch edge 0.508)
     (connect_pads (clearance 0.508))
     (min_thickness 0.254)
@@
     (polygon
       (pts
-        (xy 107.4 80.9) (xy 96.3 80.85) (xy 96.3 86.35) (xy 107.4 86.4)
+        (xy 107.4 86.3) (xy 96.3 86.35) (xy 96.3 80.85) (xy 107.4 80.8)
       )
     )
   )
-  (zone (net 0) (net_name "") (layer F.Cu) (hatch edge 0.508)
-    (connect_pads (clearance 0.508))
+  (zone (net 2) (net_name GND) (layer In2.Cu) (hatch edge 0.508)
+    (connect_pads yes (clearance 0.508))
     (min_thickness 0.254)
-    (keepout (tracks allowed) (vias not_allowed) (copperpour not_allowed))
-    (fill (arc_segments 32) (thermal_gap 0.508) (thermal_bridge_width 0.508))
+    (fill yes (arc_segments 32) (thermal_gap 0.508) (thermal_bridge_width 0.508) (smoothing fillet))
     (polygon
       (pts
-        (xy 107.4 86.3) (xy 96.3 86.35) (xy 96.3 80.85) (xy 107.4 80.8)
+        (xy 107 107) (xy 70 107) (xy 70 71) (xy 107 71)
       )
     )
